File: at101w.kicad_sch (KiCad schematic)
At the start: 286 parts, among them J2 Conn_01x04_MountingPin, Q1 Q_PMOS_GSD AO3401A, Q2 Q_NMOS_GSD 2N7002, Q3 Q_NMOS_GSD 2N7002, Q4 2N3904, SW1 SW_Push, U2 XC6206P332MR, U3 STM32F411RETx, U4 24LC64, U5 74AHCT1G125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

Commit message: fix
Parts:
- SW1: footprint random-keyboard-parts:SKQG-1155865 -> controller:switch_K2-1187SQ-A4SW-06
- U6: footprint Package_TO_SOT_SMD:SOT-666 -> Package_TO_SOT_SMD:SOT-23-6_Handsoldering
Changed lines of the file:
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@@
       (effects (font (size 1.27 1.27)) (justify left))
     )
-    (property "Footprint" "random-keyboard-parts:SKQG-1155865" (at 63.5 321.945 0)
+    (property "Footprint" "controller:switch_K2-1187SQ-A4SW-06" (at 63.5 321.945 0)
       (effects (font (size 1.27 1.27)) hide)
     )
@@
       (effects (font (size 1.27 1.27)))
     )
-    (property "Footprint" "Package_TO_SOT_SMD:SOT-666" (at 116.205 404.495 0)
-      (effects (font (size 1.27 1.27)) hide)
-    )
+    (property "Footprint" "Package_TO_SOT_SMD:SOT-23-6_Handsoldering" (at 116.205 404.495 0)
+      (effects (font (size 1.27 1.27)) hide)
+    )
